Commit message: added changes into the ur10_robotiq_set

File: ur_description/urdf/ur10_d435_robotiq_set.urdf (robot description, URDF)
Before this commit: robot ur10_arm_robotiq_set, 22 links, 21 joints
Links:
- removed link left_inner_finger
- removed link left_inner_finger_pad
- removed link left_inner_knuckle
- removed link left_outer_finger
- removed link left_outer_knuckle
- removed link right_inner_finger
- removed link right_inner_finger_pad
- removed link right_inner_knuckle
- removed link right_outer_finger
- removed link right_outer_knuckle
- removed link robotiq_arg2f_base_link
- added link robotiq_85_adapter_link; collision mesh filename=package://robotiq_2f_c2_gripper_visualization/meshes/roboti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; visual mesh filename=package://robotiq_2f_c2_gripper_visualization/meshes/roboti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
- added link robotiq_85_base_link; collision mesh filename=package://robotiq_2f_c2_gripper_visualization/meshes/roboti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; visual mesh filename=package://robotiq_2f_c2_gripper_visualization/meshes/roboti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
- added link robotiq_85_left_finger_link; collision mesh filename=package://robotiq_2f_c2_gripper_visualization/meshes/roboti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; visual mesh filename=package://robotiq_2f_c2_gripper_visualization/meshes/roboti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
- added link robotiq_85_left_finger_tip_link; collision mesh filename=package://robotiq_2f_c2_gripper_visualization/meshes/roboti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; visual mesh filename=package://robotiq_2f_c2_gripper_visualization/meshes/roboti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
- added link robotiq_85_left_inner_knuckle_link; collision mesh filename=package://robotiq_2f_c2_gripper_visualization/meshes/roboti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; visual mesh filename=package://robotiq_2f_c2_gripper_visualization/meshes/roboti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
- added link robotiq_85_left_knuckle_link; collision mesh filename=package://robotiq_2f_c2_gripper_visualization/meshes/roboti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; visual mesh filename=package://robotiq_2f_c2_gripper_visualization/meshes/roboti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
- added link robotiq_85_right_finger_link; collision mesh filename=package://robotiq_2f_c2_gripper_visualization/meshes/roboti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; visual mesh filename=package://robotiq_2f_c2_gripper_visualization/meshes/roboti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
- added link robotiq_85_right_finger_tip_link; collision mesh filename=package://robotiq_2f_c2_gripper_visualization/meshes/roboti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; visual mesh filename=package://robotiq_2f_c2_gripper_visualization/meshes/roboti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
- added link robotiq_85_right_inner_knuckle_link; collision mesh filename=package://robotiq_2f_c2_gripper_visualization/meshes/roboti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; visual mesh filename=package://robotiq_2f_c2_gripper_visualization/meshes/roboti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
- added link robotiq_85_right_knuckle_link; collision mesh filename=package://robotiq_2f_c2_gripper_visualization/meshes/roboti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; visual mesh filename=package://robotiq_2f_c2_gripper_visualization/meshes/roboti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
- added link steel_table; collision mesh filename=package://burnisher_ur10_description/meshes/collision/uap-t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; visual mesh filename=package://burnisher_ur10_description/meshes/visual/uap-tabl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
Joints:
- removed joint finger_joint
- removed joint left_inner_finger_joint
- removed joint left_inner_finger_pad_joint
- removed joint left_inner_knuckle_joint
- removed joint left_outer_finger_joint
- removed joint right_inner_finger_joint
- removed joint right_inner_finger_pad_joint
- removed joint right_inner_knuckle_joint
- removed joint right_outer_finger_joint
- removed joint right_outer_knuckle_joint
- removed joint ur10_robotiq_set_joint
- added joint robotiq_85_adapter_joint: type fixed, parent ee_link, child robotiq_85_adapter_link, origin xyz=0 0 0 rpy=0 0 0
- added joint robotiq_85_base_joint: type fixed, parent robotiq_85_adapter_link, child robotiq_85_base_link, origin xyz=.0085 0 -.0041 rpy=0 0 0, axis 1 0 0
- added joint robotiq_85_left_finger_joint: type fixed, parent robotiq_85_left_knuckle_link, child robotiq_85_left_finger_link, origin xyz=0 .00508 .03134 rpy=3.1415 0 0, axis 1 0 0, limit lower=0 upper=1.5707 effort=1000 velocity=2.0
- added joint robotiq_85_left_finger_tip_joint: type revolute, parent robotiq_85_left_inner_knuckle_link, child robotiq_85_left_finger_tip_link, origin xyz=0 .04196 -.0388 rpy=0 0 0, axis 1 0 0, limit lower=0 upper=1.5707 effort=1000 velocity=2.0, mimic joint=robotiq_85_left_knuckle_joint multiplier=-1
- added joint robotiq_85_left_inner_knuckle_joint: type revolute, parent robotiq_85_base_link, child robotiq_85_left_inner_knuckle_link, origin xyz=.04843 .0127 0 rpy=1.5707 1.5707 0, axis 1 0 0, limit lower=0 upper=1.5707 effort=1000 velocity=2.0, mimic joint=robotiq_85_left_knuckle_joint offset=0
- added joint robotiq_85_left_knuckle_joint: type revolute, parent robotiq_85_base_link, child robotiq_85_left_knuckle_link, origin xyz=.04191 .0306 0 rpy=-1.5707 1.5707 0, axis 1 0 0, limit lower=0 upper=.8575 effort=1000 velocity=2.0
- added joint robotiq_85_right_finger_joint: type fixed, parent robotiq_85_right_knuckle_link, child robotiq_85_right_finger_link, origin xyz=0 .00508 .03134 rpy=3.1415 0 0, axis 1 0 0, limit lower=0 upper=1.5707 effort=1000 velocity=2.0
- added joint robotiq_85_right_finger_tip_joint: type revolute, parent robotiq_85_right_inner_knuckle_link, child robotiq_85_right_finger_tip_link, origin xyz=0 .04196 -.0388 rpy=0 0 0, axis 1 0 0, limit lower=0 upper=1.5707 effort=1000 velocity=2.0, mimic joint=robotiq_85_left_knuckle_joint multiplier=-1
- added joint robotiq_85_right_inner_knuckle_joint: type revolute, parent robotiq_85_base_link, child robotiq_85_right_inner_knuckle_link, origin xyz=.04843 -.0127 0 rpy=-1.5707 -1.5707 0, axis 1 0 0, limit lower=0 upper=1.5707 effort=1000 velocity=2.0, mimic joint=robotiq_85_left_knuckle_joint offset=0
- added joint robotiq_85_right_knuckle_joint: type revolute, parent robotiq_85_base_link, child robotiq_85_right_knuckle_link, origin xyz=.04191 -.0306 0 rpy=1.5707 -1.5707 0, axis 1 0 0, limit lower=0 upper=1.5707 effort=1000 velocity=2.0, mimic joint=robotiq_85_left_knuckle_joint multiplier=1
- added joint steel_table_joint: type fixed, parent base_link, child steel_table, origin xyz=0.3 -0.1 0 rpy=1.570796325 0.0 0.0
