Commit message: adds the ur description with d435 and robotiq grippers
does not include all the stl files; just positioned with the gaps between

File: ur_description/urdf/ur10_arm_robotiq_set.xacro (robot description, xacro)
@@ -13,5 +13,20 @@
      <!-- robotiq (grippers) -->
     <xacro:include filename="$(find robotiq_2f_85_gripper_visualization)/urdf/robotiq_arg2f_85_model_macro.xacro"/>
-    <xacro:robotiq_arg2f_85 prefix="" connected_to="ee_link" xyz="0 0 0" rpy="0 ${pi/2} 0" />
+    <!-- <xacro:robotiq_arg2f_85 prefix="" parent="ee_link" xyz="0 0 0" rpy="0 ${pi/2} 0"/> -->
+    <xacro:robotiq_arg2f_85 prefix="" parent="d435_laser_cut_board_link" xyz="0 0 0.0224" rpy="0 0 0"/>
+    <!-- <xacro:robotiq_arg2f_85 prefix="" connected_to="ee_link" xyz="0 0 0" rpy="0 ${pi/2} 0" /> -->
+    <!-- d435 sensor -->
+  <!-- <link name="base_link" /> -->
+  <xacro:arg name="use_nominal_extrinsics" default="false"/>
+  <xacro:include filename="$(find realsense2_description)/urdf/_d435.urdf.xacro" />
+    <!-- <xacro:include filename="$(find realsense2_description)/urdf/_d435.urdf.xacro"/> -->
+  <xacro:sensor_d435 parent="d435_link" name="camera" use_nominal_extrinsics="false">
+    <origin xyz="0 0 0" rpy="0 -1.5707 3.1415"/>
+  </xacro:sensor_d435>
+    <!-- <xacro:sensor_d435 prefix="" joint_limited="false" d435_prefix="d435"/>
+    parent *origin name:=camera use_nominal_extrinsics:=false -->
+    <!-- design robotics additions and steel table -->
+    <xacro:include filename="$(find ur_description)/urdf/ur10_design_robotics_additions.xacro"/>
+    <xacro:ur10_dr_additions prefix="" joint_limited="false" d435_prefix="d435"/>
     <link name="world" />
     <joint name="world_joint" type="fixed">
